Commit message: bug fixed

File: rotors_description/urdf/crazyflie2.xacro (robot description, xacro)
@@ -35,5 +35,5 @@
   <xacro:property name="time_constant_up" value="0.0125" /> <!-- [s] -->
   <xacro:property name="time_constant_down" value="0.025" /> <!-- [s] -->
-  <xacro:property name="max_rot_velocity" value="2618" /> <!-- [rad/s] -->
+  <xacro:property name="max_rot_velocity" value="26180" /> <!-- [rad/s] -->
   <xacro:property name="rotor_drag_coefficient" value="8.06428e-05" />
   <xacro:property name="rolling_moment_coefficient" value="0.000001" />
